File: hardware/pcb/v2/v2.kicad_pcb (KiCad board)
At the start: 2 copper layers, 65.9 x 98.6 mm, 83 parts, among them J10 DF40C-30DS-0.4V, J11 XIAO-Bruecken, J12 AFC01-S24FCC-00, J13 LT7680, J14 Akku, J15 Qi, K1 Taste, K10 Taste, K11 Taste, K12 Taste, K13 Taste, K14 Taste, K15 Taste, K16 Taste, K17 Taste, K18 Taste, K19 Taste, K2 Taste, K20 Taste, K21 Taste, K22 Taste, K23 Taste, K24 Taste, K25 Taste, K26 Taste, K27 Taste, K28 Taste, K29 Taste, K3 Taste, K30 Taste, K31 Taste, K32 Taste, K33 Taste, K34 Taste, K35 Taste, K36 Taste, K37 Taste, K38 Taste, K39 Taste, K4 Taste, K40 Taste, K41 Taste, K42 Taste, K43 Taste, K44 Taste, K45 Taste, K46 Taste, K47 Taste, K48 Taste, K49 Taste, K5 Taste, K50 Taste, K6 Taste, K7 Taste, K8 Taste, K9 Taste, U1 MCP23017-E/SO, U2 LDO 2,8V (ME6211C28), U3 LDO DVDD (pruefen)

Commit message: Hauptplatine V2: verdrahtet (Freerouting), DRC ohne Fehler, Vorschau
Co-Authored-By: Claude Opus 5.5 <noreply@anthropic.com>
Claude-Session: https://claude.ai/code/session_018xurYUYAMjcQd5yu9g7cvN
Routing:
- net GND: track 0.00 -> 225.5 mm, vias 0 -> 4
- net 3V3: track 0.00 -> 146.1 mm, vias 0 -> 2
- net C5: track 0.00 -> 141.4 mm, vias 0 -> 3
- net R8: track 0.00 -> 126.8 mm, vias 0 -> 6
- net C4: track 0.00 -> 119.4 mm, vias 0 -> 1
- net C0: track 0.00 -> 118.4 mm, vias 0 -> 1
- net R4: track 0.00 -> 115.8 mm, vias 0 -> 8
- net R0: track 0.00 -> 115.3 mm, vias 0 -> 7
- net R7: track 0.00 -> 114.4 mm, vias 0 -> 6
- net C1: track 0.00 -> 103.8 mm, vias 0 -> 1
- net R6: track 0.00 -> 102.4 mm, vias 0 -> 6
- net R5: track 0.00 -> 95.6 mm, vias 0 -> 7
- net C2: track 0.00 -> 92.5 mm, vias 0 -> 2
- net C3: track 0.00 -> 89.4 mm, vias 0 -> 2
- net R1: track 0.00 -> 84.4 mm, vias 0 -> 7
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Other:
- board text added: "XIAO (USB oben)"
- board text removed: "XIAO ESP32S3 (Unterseite zur Platine, USB oben)"
